File: USBPD.kicad_sch (KiCad schematic)
At the start: 22 parts, among them J1 Conn_01x10, J2 USB_C_Receptacle_USB2.0, J3 Conn_01x04, J4 Conn_01x02, SW1 SW_Push, U1 FUSB302BMPX

Commit message: change 100nF to 470pf
Parts:
- C4, C6: value 100n -> 470p
Changed lines of the file:
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@@
       (effects (font (size 1.27 1.27)) (justify left))
     )
-    (property "Value" "100n" (id 1) (at 93.091 89.5862 0)
+    (property "Value" "470p" (id 1) (at 93.091 89.5862 0)
       (effects (font (size 1.27 1.27)) (justify left))
     )
@@
       (effects (font (size 1.27 1.27)) (justify left))
     )
-    (property "Value" "100n" (id 1) (at 108.585 89.5862 0)
+    (property "Value" "470p" (id 1) (at 108.585 89.5862 0)
       (effects (font (size 1.27 1.27)) (justify left))
     )
@@
     )
     (path "/3c861525-bffa-4f66-a992-362db2d7daca"
-      (reference "C4") (unit 1) (value "100n") (footprint "Capacitor_SMD:C_0603_1608Metric")
+      (reference "C4") (unit 1) (value "470p") (footprint "Capacitor_SMD:C_0603_1608Metric")
     )
     (path "/daa2f944-b48f-4e1d-a28d-4efcadad7bdd"
-      (reference "C6") (unit 1) (value "100n") (footprint "Capacitor_SMD:C_0603_1608Metric")
+      (reference "C6") (unit 1) (value "470p") (footprint "Capacitor_SMD:C_0603_1608Metric")
     )
     (path "/284abe0f-35f5-43e9-ba6c-4aa6f2e56eae"
